Commit message: controllers updated

File: rotf_control/urdf/model_1.urdf (robot description, URDF)
Before this commit: robot diff_bot, 3 links, 2 joints
Links:
- added link laser, mass 0.2; visual cylinder length=0.1 radius=0.001
Joints:
- added joint laser_joint: type fixed, parent base_link, child laser, origin xyz=0 0 0.1 rpy=0 0 0

Commit message: controllers updated

File: rotf_control/urdf/model_1.urdf (robot description, URDF)
Before this commit: robot diff_bot, 4 links, 3 joints
Joints:
- joint right_wheel_joint: limit effort=100 velocity=100 -> effort=10 velocity=10
