Commit message: teb changes

File: rotf_control/urdf/model.urdf (robot description, URDF)
Before this commit: robot diff_bot, 4 links, 3 joints
Links:
- added link base_footprint
- link base_link: mass 15 -> 10.0; geometry collision box size=.4 .2 .1; collision sphere radius=0.05
- link left_wheel: mass 1 -> 5; geometry collision cylinder length=0.05 radius=0.1; visual cylinder length=0.05 radius=0.1
- link right_wheel: mass 1 -> 5; geometry collision cylinder length=0.05 radius=0.1; visual cylinder length=0.05 radius=0.1
Joints:
- added joint base_footprint_to_base_link: type fixed, parent base_footprint, child base_link, origin xyz=0.0 0.0 0.0 rpy=0.0 0.0 0.0, axis 0.0 0.0 0.1
- joint laser_joint: origin xyz=0 0 0.12 rpy=0 0 0 -> xyz=0 0 0.1 rpy=0 0 0
- joint left_wheel_joint: axis 0.0 1.0 0.0 -> 0 1 0; limit effort=100.0 velocity=100.0 -> effort=100 velocity=100; origin xyz=-0.15 -0.15 0.0 rpy=0.0 0.0 0.0 -> xyz=0.1 0.15 0 rpy=0 0 0
- joint right_wheel_joint: axis 0.0 1.0 0.0 -> 0 1 0; limit effort=100.0 velocity=100.0 -> effort=10 velocity=10; origin xyz=-0.15 0.15 0.0 rpy=0.0 0.0 0.0 -> xyz=0.1 -0.15 0 rpy=0 0 0

Commit message: localisation is changed

File: rotf_control/urdf/model.urdf (robot description, URDF)
Before this commit: robot diff_bot, 5 links, 4 joints
Links:
- removed link base_footprint
Joints:
- removed joint base_footprint_to_base_link

File: rotf_control/urdf/model_1.urdf (robot description, URDF)
Before this commit: robot diff_bot, 4 links, 3 joints
Joints:
- joint right_wheel_joint: limit effort=10 velocity=10 -> effort=100 velocity=100
